File: ESP32_Bluetooth_Speaker/ESP32_Bluetooth_Speaker.kicad_sch (KiCad schematic)
At the start: 0 parts

Commit message: Started Schematic capture for PCB.
Parts:
- added U1: ESP32-WROOM-32, Speaker_Lib:ESP32_30pin, symbol RF_Module:ESP32-WROOM-32
Connections:
- new net: U1.1 (GND), U1.15 (GND), U1.38 (GND), U1.39 (GND)
Changed lines of the file:
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@@
 	(generator_version "9.0")
 	(paper "A4")
+	(symbol
+		(lib_id "RF_Module:ESP32-WROOM-32")
+		(at 144.78 91.44 0)
+		(unit 1)
+		(exclude_from_sim no)
+		(in_bom yes)
+		(on_board yes)
+		(dnp no)
+		(fields_autoplaced yes)
+		(property "Reference" "U1"
+			(at 146.9233 53.34 0)
+			(effects
+				(font
+					(size 1.27 1.27)
+				)
+				(justify left)
+			)
+		)
+		(property "Value" "ESP32-WROOM-32"
+			(at 146.9233 55.88 0)
+			(effects
+				(font
+					(size 1.27 1.27)
+				)
+				(justify left)
+			)
+		)
+		(property "Footprint" "Speaker_Lib:ESP32_30pin"
+			(at 144.78 129.54 0)
+			(effects
+				(font
+					(size 1.27 1.27)
+				)
+				(hide yes)
+			)
+		)
+		(property "Datasheet" "https://www.espressif.com/sites/default/files/documentation/esp32-wroom-32_datasheet_en.pdf"
+			(at 137.16 90.17 0)
+			(effects
+				(font
+					(size 1.27 1.27)
+				)
+				(hide yes)
+			)
+		)
+		(property "Description" "RF Module, ESP32-D0WDQ6 SoC, Wi-Fi 802.11b/g/n, Bluetooth, BLE, 32-bit, 2.7-3.6V, onboard antenna, SMD"
+			(at 144.78 91.44 0)
+			(effects
+				(font
+					(size 1.27 1.27)
+				)
+				(hide yes)
+			)
+		)
+		(pin "22"
+		)
+		(pin "7"
+		)
+		(pin "9"
+		)
+		(pin "6"
+		)
+		(pin "38"
+		)
+		(pin "35"
+		)
+		(pin "4"
+		)
+		(pin "18"
+		)
+		(pin "37"
+		)
+		(pin "28"
+		)
+		(pin "29"
+		)
+		(pin "27"
+		)
+		(pin "23"
+		)
+		(pin "10"
+		)
+		(pin "8"
+		)
+		(pin "12"
+		)
+		(pin "14"
+		)
+		(pin "2"
+		)
+		(pin "36"
+		)
+		(pin "13"
+		)
+		(pin "16"
+		)
+		(pin "19"
+		)
+		(pin "32"
+		)
+		(pin "11"
+		)
+		(pin "39"
+		)
+		(pin "15"
+		)
+		(pin "1"
+		)
+		(pin "5"
+		)
+		(pin "3"
+		)
+		(pin "21"
+		)
+		(pin "24"
+		)
+		(pin "26"
+		)
+		(pin "25"
+		)
+		(pin "17"
+		)
+		(pin "34"
+		)
+		(pin "33"
+		)
+		(pin "30"
+		)
+		(pin "31"
+		)
+		(pin "20"
+		)
+		(instances
+			(project ""
+				(path "/c33c675d-3eda-4279-b4bc-97e4f921166c"
+					(reference "U1")
+					(unit 1)
+				)
+			)
+		)
+	)
 	(sheet_instances
 		(path "/"

Commit message: Initial Commit for Project
Parts:
- removed U1: ESP32-WROOM-32, Speaker_Lib:ESP32_30pin, symbol RF_Module:ESP32-WROOM-32
- added C1, C2: 47pF, Capacitor_SMD:C_0805_2012Metric, symbol Device:C_Small
- added C10, C6, C7: 47uF, Capacitor_SMD:CP_Elec_6.3x5.4, symbol Device:C_Polarized_Small_US
- added C11, C12, C3, C4, C5, C8, C9: 0.1uF, Capacitor_SMD:C_0805_2012Metric, symbol Device:C_Small
- added C13, C14: 220pF, Capacitor_SMD:C_0805_2012Metric, symbol Device:C_Small
- added D1: POWER (RED), LED_SMD:LED_0805_2012Metric, symbol Device:LED
- added J1: USB_B_Mini, Connector_USB:USB_Mini-B_Wuerth_65100516121_Horizontal, symbol Connector:USB_B_Mini
- added J2: POWER INPUT, Connector_BarrelJack:BarrelJack_CUI_PJ-102AH_Horizontal, symbol Connector:Barrel_Jack_Switch_Pin3Ring
- added J3: SPEAKER, TerminalBlock_RND:TerminalBlock_RND_205-00232_1x02_P5.08mm_Horizontal, symbol Connector:Screw_Terminal_01x02
- added Q1, Q2: MMBT3904, Package_TO_SOT_SMD:SOT-23, symbol Transistor_BJT:MMBT3904
- added R1, R12, R2, R3, R4, R7, R8, R9: 10k, Resistor_SMD:R_0805_2012Metric, symbol Device:R_US
- added R10, R11, R13, R14: 330, Resistor_SMD:R_0805_2012Metric, symbol Device:R_US
- added R15: 1M, Resistor_SMD:R_0805_2012Metric, symbol Device:R_US
- added R5, R6: 27, Resistor_SMD:R_0805_2012Metric, symbol Device:R_US
- added RX1: (GREEN), LED_SMD:LED_0805_2012Metric, symbol Device:LED
- added SW1: PAUSE, Button_Switch_THT:SW_Tactile_SPST_Angled_PTS645Vx58-2LFS, symbol Switch:SW_Push
- added SW2: PREV, Button_Switch_THT:SW_Tactile_SPST_Angled_PTS645Vx58-2LFS, symbol Switch:SW_Push
- added SW3: NEXT, Button_Switch_THT:SW_Tactile_SPST_Angled_PTS645Vx58-2LFS, symbol Switch:SW_Push
- added SW4: V+, Button_Switch_THT:SW_Tactile_SPST_Angled_PTS645Vx58-2LFS, symbol Switch:SW_Push
- added SW5: V-, Button_Switch_THT:SW_Tactile_SPST_Angled_PTS645Vx58-2LFS, symbol Switch:SW_Push
- added SW6: RESET, Alarm_Clock_Lib:SKQYAAE010, symbol Switch:SW_Push
- added TX1: (AMBER), LED_SMD:LED_0805_2012Metric, symbol Device:LED
- added U1: FT231XS, Package_SO:SSOP-20_3.9x8.7mm_P0.635mm, symbol Interface_USB:FT231XS
- added U2: ESP32-WROOM-32E, RF_Module:ESP32-WROOM-32D, symbol RF_Module:ESP32-WROOM-32E
- added U3: NCP1117, Package_TO_SOT_SMD:TO-252-2, symbol Regulator_Linear:LM317_TO-252
- added U4: MAX98357A, Package_DFN_QFN:TQFN-16-1EP_3x3mm_P0.5mm_EP1.23x1.23mm, symbol Audio:MAX98357A
- added USER1: (RED), LED_SMD:LED_0805_2012Metric, symbol Device:LED
Connections:
- new net: Q2.1 (B), R3.2
- new net: C14.1, J3.1 (Pin_1), U4.9 (OUTP)
- new net: C13.1, J3.2 (Pin_2), U4.10 (OUTN)
- new net: R15.2, U4.4 (~{SD_MODE})
- new net: Q1.1 (B), R2.2
- new net: D1.2 (A), R14.1
- new net: RX1.1 (K), U1.17 (CBUS1)
- new net: R10.1, RX1.2 (A)
- new net: R13.1, USER1.2 (A)
- new net: C2.1, J1.2 (D-), R6.1
- new net: C1.1, J1.3 (D+), R5.1
- new net: TX1.1 (K), U1.10 (CBUS2)
- new net: R5.2, U1.11 (USBDP)
- new net: R6.2, U1.12 (USBDM)
- new net: R11.1, TX1.2 (A)
- new net: U2.30 (IO18), USER1.1 (K)
- new net +3V3: C10.1, C11.1, C12.1, C3.1, R1.2, R10.2, R11.2, R12.2, R13.2, R14.2, R4.2, R7.2, R8.2, R9.2, U1.13 (3V3OUT), U1.14 (~{RESET}), U1.15 (VCC), U1.3 (VCCIO), U2.2 (VDD), U3.2 (VO)
- new net +5V: C6.1, C7.1, C8.1, J2.1, R15.1, U3.3 (VI), U4.7 (VDD), U4.8 (VDD)
- new net BCLK: U2.12 (IO27), U4.16 (BCLK)
- new net DIN: U2.11 (IO26), U4.1 (DIN)
- new net DTR: Q1.2 (E), R3.1, U1.1 (~{DTR})
- new net EN: C5.2, C9.1, Q2.3 (C), R12.1, SW6.2, U2.3 (EN)
- new net GND: C1.2, C10.2, C11.2, C12.2, C13.2, C14.2, C2.2, C3.2, C4.2, C5.1, C6.2, C7.2, C8.2, C9.2, D1.1 (K), J1.5 (GND), J1.6 (Shield), J2.2, J2.3, SW1.2, SW2.2, SW3.2, SW4.2, SW5.2, SW6.1, U1.16 (GND), U1.6 (GND), U2.1 (GND), U2.15 (GND), U2.38 (GND), U2.39 (GND), U3.1 (ADJ), U4.11 (GND), U4.15 (GND), U4.3 (GND)
- new net GPIO0: C4.1, Q1.3 (C), U2.25 (IO0)
- new net LRCLK: U2.13 (IO14), U4.14 (LRCLK)
- new net PB1: R1.1, SW1.1, U2.29 (IO5)
- new net PB2: R4.1, SW2.1, U2.31 (IO19)
- new net PB3: R7.1, SW3.1, U2.33 (IO21)
- new net PB4: R8.1, SW4.1, U2.36 (IO22)
- new net PB5: R9.1, SW5.1, U2.37 (IO23)
- new net RTS: Q2.2 (E), R2.1, U1.2 (~{RTS})
- new net RXD: U1.4 (RXD), U2.35 (TXD0/IO1)
- new net TXD: U1.20 (TXD), U2.34 (RXD0/IO3)
- no-connect marks 0 -> 24
Other:
- note added: "MAX98357A Layout"
- note added: "Power and Decoupling"
- note added: "Reset and Bootloader Control"
- note added: "USB Interface"
- note added: "User Interface"
