File: ESP32_Bluetooth_Speaker/ESP32_Bluetooth_Speaker_devpcb/ESP32_Bluetooth_Speaker_devpcb.kicad_pcb (KiCad board)
At the start: 2 copper layers, 53.3 x 68.6 mm, 18 parts, among them J1 POWER INPUT, SW1 PAUSE, SW2 PREV, SW3 NEXT, SW4 V+, SW5 V-, U1 ESP32_DevKit_V1_DOIT

Commit message: Added CAD assembly and surface mount PCB initial rev
Parts:
- moved C1 8.12 mm to (140.5, 83.2), turned to -90 degrees
- moved C2 2.69 mm to (163.8, 138.5)
- moved R6 1.49 mm to (160.3, 131.8)
Routing:
- net +5V: track 126.4 -> 102.8 mm
- net Net-(D1-A): track 13.8 -> 12.3 mm
- added copper zone on F.Cu, net +5V
